File: TE0724_Connector.kicad_sch (KiCad schematic)
At the start: 1 part, among them J1 SS5-80-3.50-X-D-K-XX

Commit message: BOM update
completed the BOM list
Parts:
- J1: MANUFACTURER_PART_NUMBER (none) -> SS5-80-3.50-L-D-K-TR
Changed lines of the file:
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@@
+			)
+		)
+		(property "MANUFACTURER_PART_NUMBER" "SS5-80-3.50-L-D-K-TR "
+			(at 97.79 80.01 0)
+			(effects
+				(font
+					(size 1.27 1.27)
+				)
+				(hide yes)
 			)
 		)
